File: RJ45AnalogEagle/RJ45AnalogEagle.brd (EAGLE design)
At the start: 32 x 28 mm, 4 parts

Commit message: modified design
Connections:
- net N$3 renamed AIN2
- net N$4 renamed GPIO
- net N$5 renamed AIN1
- net N$6 renamed AIN3
Changed lines of the file:
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@@
 <layer number="17" name="Pads" color="2" fill="1" visible="yes" active="yes"/>
 <layer number="18" name="Vias" color="2" fill="1" visible="no" active="yes"/>
-<layer number="19" name="Unrouted" color="6" fill="1" visible="no" active="yes"/>
+<layer number="19" name="Unrouted" color="6" fill="1" visible="yes" active="yes"/>
 <layer number="20" name="Dimension" color="15" fill="1" visible="yes" active="yes"/>
 <layer number="21" name="tPlace" color="7" fill="1" visible="no" active="yes"/>
@@
 <contactref element="U$1" pad="1"/>
 </signal>
-<signal name="N$3">
+<signal name="AIN2">
 <contactref element="U$1" pad="4"/>
 <contactref element="U$2" pad="4"/>
@@
 <wire x1="15.365" y1="15.7206" x2="15.365" y2="16.11" width="0.8128" layer="1"/>
 </signal>
-<signal name="N$4">
+<signal name="GPIO">
 <contactref element="U$1" pad="6"/>
 <contactref element="U$2" pad="6"/>
@@
 <wire x1="17.905" y1="15.8476" x2="17.905" y2="16.11" width="0.8128" layer="1"/>
 </signal>
-<signal name="N$5">
+<signal name="AIN1">
 <contactref element="U$1" pad="3"/>
 <contactref element="U$2" pad="1"/>
@@
 <wire x1="9.905" y1="17" x2="11.555" y2="18.65" width="0.8128" layer="1"/>
 </signal>
-<signal name="N$6">
+<signal name="AIN3">
 <contactref element="U$1" pad="5"/>
 <contactref element="U$2" pad="7"/>
