File: RJ45AnalogEagle/RJ45AnalogEagle.sch (EAGLE design)
At the start: 2 parts

Commit message: modified design
Connections:
- net N$3 renamed AIN2
- net N$4 renamed GPIO
- net N$5 renamed AIN1
- net N$6 renamed AIN3
Changed lines of the file:
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@@
 </segment>
 </net>
-<net name="N$3" class="0">
+<net name="AIN2" class="0">
 <segment>
 <pinref part="U$1" gate="X" pin="4"/>
@@
 </segment>
 </net>
-<net name="N$4" class="0">
+<net name="GPIO" class="0">
 <segment>
 <pinref part="U$1" gate="X" pin="6"/>
@@
 </segment>
 </net>
-<net name="N$5" class="0">
+<net name="AIN1" class="0">
 <segment>
 <pinref part="U$1" gate="X" pin="3"/>
@@
 </segment>
 </net>
-<net name="N$6" class="0">
+<net name="AIN3" class="0">
 <segment>
 <pinref part="U$1" gate="X" pin="5"/>
